File: Hardware/TRV_MRF49_U_V1.1_F.brd (EAGLE design)
At the start: 40 x 28 mm, 38 parts, among them IC1 MRF49XA, IC2 MEGA168PA-AU, IC3 LP2992-IM5-3.3, Q1 IRLML9301, X1 ANT, X2 GND, X3 GND, X4 GND, X5 GND

Commit message: Added PDF View
Parts:
- EXT: device Conn:ML20 -> Conn:ML20S
- ISP: device Conn:ML6 -> Conn:ML6S
Changed lines of the file:
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@@
 <setting verticaltext="up"/>
 </settings>
-<grid distance="1.27" unitdist="mm" unit="mm" style="lines" multiple="1" display="yes" altdistance="0.025" altunitdist="inch" altunit="inch"/>
+<grid distance="1" unitdist="mm" unit="mm" style="lines" multiple="1" display="yes" altdistance="0.025" altunitdist="inch" altunit="inch"/>
 <layers>
-<layer number="1" name="Top" color="4" fill="1" visible="yes" active="yes"/>
+<layer number="1" name="Top" color="4" fill="1" visible="no" active="yes"/>
 <layer number="2" name="Route2" color="1" fill="3" visible="no" active="no"/>
 <layer number="3" name="Route3" color="4" fill="3" visible="no" active="no"/>
@@
 <layer number="14" name="Route14" color="1" fill="6" visible="no" active="no"/>
 <layer number="15" name="Route15" color="4" fill="6" visible="no" active="no"/>
-<layer number="16" name="Bottom" color="1" fill="1" visible="yes" active="yes"/>
-<layer number="17" name="Pads" color="2" fill="1" visible="yes" active="yes"/>
-<layer number="18" name="Vias" color="2" fill="1" visible="yes" active="yes"/>
-<layer number="19" name="Unrouted" color="6" fill="1" visible="yes" active="yes"/>
+<layer number="16" name="Bottom" color="1" fill="1" visible="no" active="yes"/>
+<layer number="17" name="Pads" color="2" fill="1" visible="no" active="yes"/>
+<layer number="18" name="Vias" color="2" fill="1" visible="no" active="yes"/>
+<layer number="19" name="Unrouted" color="6" fill="1" visible="no" active="yes"/>
 <layer number="20" name="Dimension" color="15" fill="1" visible="yes" active="yes"/>
-<layer number="21" name="tPlace" color="7" fill="1" visible="no" active="yes"/>
+<layer number="21" name="tPlace" color="7" fill="1" visible="yes" active="yes"/>
 <layer number="22" name="bPlace" color="7" fill="1" visible="no" active="yes"/>
-<layer number="23" name="tOrigins" color="15" fill="1" visible="yes" active="yes"/>
+<layer number="23" name="tOrigins" color="15" fill="1" visible="no" active="yes"/>
 <layer number="24" name="bOrigins" color="15" fill="1" visible="no" active="yes"/>
-<layer number="25" name="tNames" color="7" fill="1" visible="no" active="yes"/>
+<layer number="25" name="tNames" color="7" fill="1" visible="yes" active="yes"/>
 <layer number="26" name="bNames" color="7" fill="1" visible="no" active="yes"/>
-<layer number="27" name="tValues" color="7" fill="1" visible="no" active="yes"/>
+<layer number="27" name="tValues" color="7" fill="1" visible="yes" active="yes"/>
 <layer number="28" name="bValues" color="7" fill="1" visible="no" active="yes"/>
 <layer number="29" name="tStop" color="7" fill="3" visible="no" active="yes"/>
-<layer number="30" name="bStop" color="7" fill="6" visible="yes" active="yes"/>
+<layer number="30" name="bStop" color="7" fill="6" visible="no" active="yes"/>
 <layer number="31" name="tCream" color="7" fill="4" visible="no" active="yes"/>
 <layer number="32" name="bCream" color="7" fill="5" visible="no" active="yes"/>
@@
 <layer number="45" name="Holes" color="7" fill="1" visible="no" active="yes"/>
 <layer number="46" name="Milling" color="3" fill="1" visible="no" active="yes"/>
-<layer number="47" name="Measures" color="7" fill="1" visible="yes" active="yes"/>
+<layer number="47" name="Measures" color="7" fill="1" visible="no" active="yes"/>
 <layer number="48" name="Document" color="7" fill="1" visible="no" active="yes"/>
 <layer number="49" name="Reference" color="7" fill="1" visible="no" active="yes"/>
@@
 <wire x1="0" y1="0" x2="40" y2="0" width="0" layer="20"/>
 <wire x1="40" y1="0" x2="40" y2="28" width="0" layer="20"/>
-<wire x1="40" y1="28" x2="0" y2="28" width="0" layer="20"/>
 <wire x1="0" y1="28" x2="0" y2="0" width="0" layer="20"/>
 <hole x="36.5" y="24.5" drill="3.2"/>
@@
 <text x="29.845" y="26.416" size="1.27" layer="1" font="vector" ratio="15">TOP</text>
 <text x="33.02" y="26.416" size="1.27" layer="16" font="vector" ratio="15" rot="MR0">BOT</text>
+<wire x1="0" y1="28" x2="40" y2="28" width="0" layer="20"/>
 </plain>
 <attributes>
@@
 <element name="IC2" library="atmel" package="TQFP32-08" value="MEGA168PA-AU" x="14.224" y="14.986" rot="R45"/>
 <element name="C5" library="RCL" package="0603" value="100n" x="19.304" y="19.304" rot="R270"/>
-<element name="ISP" library="Conn" package="ML6" value="ISP" x="22.86" y="24.13" rot="R180"/>
+<element name="ISP" library="Conn" package="ML6S" value="ISP" x="22.86" y="24.13" smashed="yes" rot="R180">
+<attribute name="VALUE" x="16.129" y="26.289" size="1.778" layer="27" ratio="10" rot="R270"/>
+</element>
 <element name="C8" library="RCL" package="0603" value="100n" x="20.701" y="19.304" rot="R270"/>
 <element name="C9" library="RCL" package="0603" value="100n" x="9.144" y="10.4648" rot="R45"/>
@@
 <element name="LED1" library="Optic" package="0603" value="LEDR" x="22.733" y="8.382" rot="R90"/>
 <element name="R1" library="RCL" package="0603" value="10k" x="24.13" y="8.382" rot="R90"/>
-<element name="EXT" library="Conn" package="ML20" value="EXT" x="3.81" y="13.97" rot="R270"/>
+<element name="EXT" library="Conn" package="ML20S" value="EXT" x="3.81" y="13.97" rot="R270"/>
 <element name="L1" library="RCL" package="0603" value="100nH" x="33.147" y="17.272" rot="R270"/>
 <element name="L2" library="RCL" package="0603" value="8.2nH" x="33.147" y="14.605" rot="R90"/>
@@
 <element name="R3" library="RCL" package="0603" value="0R" x="15.24" y="2.54"/>
 <element name="DS1" library="Diode" package="SOD323" value="PESD12VL1BA" x="18.415" y="2.54"/>
-<element name="X6" library="Conn" package="S1.27R" value="" x="23.622" y="12.065"/>
+<element name="X6" library="Conn" package="S1.27R" value="" x="23.622" y="12.065" smashed="yes">
+<attribute name="NAME" x="23.241" y="11.811" size="0.4064" layer="25"/>
+</element>
 <element name="QR1" library="QUARTZ" package="CR" value="8M" x="11.684" y="8.382" rot="R135"/>
 <element name="R4" library="RCL" package="0603" value="n.b." x="21.336" y="6.858" rot="R90"/>
