File: Hardware/TRV_MRF49_U_V1.1_F.sch (EAGLE design)
At the start: 38 parts, among them IC1 MRF49XA, IC2 MEGA168PA-AU, IC3 LP2992-IM5-3.3, Q1 IRLML9301, X1 ANT, X2 GND, X3 GND, X4 GND, X5 GND

Commit message: Added PDF View
Parts:
- EXT: device Conn:ML20E -> Conn:ML20SE
- ISP: device Conn:ML6E -> Conn:ML6ES
- QM1: device QUARTZ:QMABM3C -> QUARTZ:QM5X3.2
Changed lines of the file:
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@@
 <part name="C5" library="RCL" deviceset="C" device="0603" value="100n"/>
 <part name="GND8" library="supply1" deviceset="GND" device=""/>
-<part name="ISP" library="Conn" deviceset="ML6E" device="" value="ISP"/>
+<part name="ISP" library="Conn" deviceset="ML6E" device="S" value="ISP"/>
 <part name="GND9" library="supply1" deviceset="GND" device=""/>
 <part name="C8" library="RCL" deviceset="C" device="0603" value="100n"/>
@@
 <part name="+3V7" library="supply1" deviceset="+3V3" device=""/>
 <part name="+3V8" library="supply1" deviceset="+3V3" device=""/>
-<part name="EXT" library="Conn" deviceset="ML20?E" device="" value="EXT"/>
+<part name="EXT" library="Conn" deviceset="ML20?E" device="S" value="EXT"/>
 <part name="L1" library="RCL" deviceset="L" device="0603" value="100nH"/>
 <part name="L2" library="RCL" deviceset="L" device="0603" value="8.2nH"/>
@@
 <part name="QR1" library="QUARTZ" deviceset="QR" device="CR" value="8M"/>
 <part name="R4" library="RCL" deviceset="R" device="0603" value="n.b."/>
-<part name="QM1" library="QUARTZ" deviceset="QM" device="ABM3C" value="10M"/>
+<part name="QM1" library="QUARTZ" deviceset="QM" device="5X3.2" value="10M"/>
 <part name="C2" library="RCL" deviceset="C_POL" device="SMCB" value="10u"/>
 <part name="GND20" library="supply1" deviceset="GND" device=""/>
